File: Transmitter_11-16.sch (EAGLE design)
At the start: 23 parts, among them IC1 7805T, IC2 REG1117, IC3 HT12E", M2 WIRELESS-XY-FST#V, Q1 16MHz, U1 328P

Commit message: Add files via upload
Parts:
- renumbered IC1 to V_REG_5, IC2 to V_REG_3.3, IC3 to ENCODER, JP1 to BATTERY, M2 to 433HMZ_TX, U1 to ATMEGA_328
Other:
- note added: "11/16/17"
- note added: "TEAM 4 Gomathy Krishna, Mark Kaldas, Tapas Sastry, Yebin Woo"
- note added: "Transmitter Side of Hand Gesture Controlled Robot"
- note added: "Ver.2"
- note removed: "3.3V V-Reg"
- note removed: "433MHzTransmitter"
- note removed: "Atmel Atmega 328"
- note removed: "Battery"
- note removed: "HT12E Encoder"
- note removed: "Transmitter of Hand Gesture Controlled Robot (Team 4)"
