File: Reciever_11-16.sch (EAGLE design)
At the start: 23 parts, among them IC1 HT12D", IC2 L293D, IC3 7805T, M1 WIRELESS-XY-MK-5V-V

Commit message: Add files via upload
Parts:
- renumbered IC1 to DECODER, IC2 to DRIVER_IC, IC3 to V_REG, JP1 to MOTOR1, JP2 to MOTOR2, M1 to 433MHZ_RX
Other:
- note added: "11/16/17"
- note added: "Receiver Side of Hand Gesture Controlled Robot"
- note added: "TEAM 4 Gomathy Krishna, Mark Kaldas, Tapas Sastry, Yebin Woo"
- note added: "Ver.2"
- note removed: "433MHz Receiver"
- note removed: "HT12D Decoder"
- note removed: "L293D Driver IC"
- note removed: "Power Supply"
- note removed: "Receiver side of Hand Gesture controlled Robot (Team 4)"
