File: Reciever_11-16.brd (EAGLE design)
At the start: 35.5 x 70.8 mm, 23 parts, among them IC1 HT12D", IC2 L293D, IC3 7805T, M1 WIRELESS-XY-MK-5V-V

Commit message: Add files via upload
Parts:
- renumbered JP1 to MOTOR1, JP2 to MOTOR2
Changed lines of the file:
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@@
 <wire x1="35.54" y1="70.79" x2="0" y2="70.79" width="0" layer="20"/>
 <wire x1="0" y1="70.79" x2="0" y2="0" width="0" layer="20"/>
-<text x="34.29" y="26.67" size="1.778" layer="1" font="vector" ratio="15" rot="R90">Team 04</text>
-<text x="13.97" y="26.67" size="1.778" layer="16" font="vector" ratio="15" rot="MR90">Team 04</text>
+<text x="16.51" y="26.67" size="1.778" layer="21" font="vector" ratio="15" rot="MR90">Team 04</text>
 </plain>
 <attributes>
@@
 <element name="R4" library="adafruit" library_urn="urn:adsk.eagle:library:420" package="R0805" value="220" x="20.32" y="10.16"/>
 <element name="R5" library="adafruit" library_urn="urn:adsk.eagle:library:420" package="R0805" value="220" x="25.4" y="13.97"/>
-<element name="JP1" library="pinhead" library_urn="urn:adsk.eagle:library:325" package="1X02" package3d_urn="urn:adsk.eagle:package:22435/2" value="" x="3.81" y="3.81" rot="R180"/>
-<element name="JP2" library="pinhead" library_urn="urn:adsk.eagle:library:325" package="1X02" package3d_urn="urn:adsk.eagle:package:22435/2" value="" x="31.75" y="3.81" rot="R180"/>
+<element name="MOTOR1" library="pinhead" library_urn="urn:adsk.eagle:library:325" package="1X02" package3d_urn="urn:adsk.eagle:package:22435/2" value="" x="3.81" y="3.81" rot="R180"/>
+<element name="MOTOR2" library="pinhead" library_urn="urn:adsk.eagle:library:325" package="1X02" package3d_urn="urn:adsk.eagle:package:22435/2" value="" x="31.75" y="3.81" rot="R180"/>
 <element name="C1" library="adafruit" library_urn="urn:adsk.eagle:library:420" package="C0805" value="0.1u" x="6.35" y="24.13"/>
 <element name="C2" library="adafruit" library_urn="urn:adsk.eagle:library:420" package="C0805" value="10u" x="22.86" y="57.15" rot="R90"/>
@@
 <signal name="-RIGHT" class="2">
 <contactref element="IC2" pad="11"/>
-<contactref element="JP2" pad="2"/>
+<contactref element="MOTOR2" pad="2"/>
 <wire x1="26.67" y1="24.13" x2="29.21" y2="24.13" width="1.27" layer="16"/>
 <wire x1="26.67" y1="7.62" x2="26.67" y2="24.13" width="1.27" layer="16"/>
@@
 <signal name="+RIGHT" class="2">
 <contactref element="IC2" pad="14"/>
-<contactref element="JP2" pad="1"/>
+<contactref element="MOTOR2" pad="1"/>
 <wire x1="33.655" y1="31.75" x2="29.21" y2="31.75" width="1.27" layer="16"/>
 <wire x1="33.655" y1="5.08" x2="33.655" y2="31.75" width="1.27" layer="16"/>
@@
 <signal name="-LEFT" class="2">
 <contactref element="IC2" pad="6"/>
-<contactref element="JP1" pad="1"/>
+<contactref element="MOTOR1" pad="1"/>
 <wire x1="13.335" y1="24.13" x2="21.59" y2="24.13" width="1.27" layer="16"/>
 <wire x1="13.335" y1="12.065" x2="13.335" y2="24.13" width="1.27" layer="16"/>
@@
 <signal name="+LEFT" class="2">
 <contactref element="IC2" pad="3"/>
-<contactref element="JP1" pad="2"/>
+<contactref element="MOTOR1" pad="2"/>
 <wire x1="20.955" y1="31.115" x2="21.59" y2="31.75" width="1.27" layer="1"/>
 <wire x1="19.05" y1="31.115" x2="20.955" y2="31.115" width="1.27" layer="1"/>

Commit message: Add files via upload
Routing:
- net GND: vias 1 -> 12
- added copper zone on layer 1, net GND
- removed copper zone on layer 1, net N$15
Other:
- board text added: "Team 04 Ver.2"
- board text removed: "Team 04"
Changed lines of the file:
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@@
 <wire x1="35.54" y1="70.79" x2="0" y2="70.79" width="0" layer="20"/>
 <wire x1="0" y1="70.79" x2="0" y2="0" width="0" layer="20"/>
-<text x="16.51" y="26.67" size="1.778" layer="21" font="vector" ratio="15" rot="MR90">Team 04</text>
+<text x="16.51" y="36.83" size="1.27" layer="21" font="vector" ratio="15" rot="MR270">Team 04
+Ver.2</text>
 </plain>
 <attributes>
@@
 <wire x1="27.94" y1="47.625" x2="27.94" y2="47.84" width="0.1778" layer="1"/>
 <via x="12.065" y="24.13" extent="1-16" drill="0.4064"/>
-</signal>
-<signal name="N$15">
 <polygon width="0.2" layer="1">
 <vertex x="0" y="71.12"/>
@@
 <vertex x="0" y="0"/>
 </polygon>
+<via x="10.16" y="55.88" extent="1-16" drill="0.45"/>
+<via x="33.02" y="46.99" extent="1-16" drill="0.45"/>
+<via x="21.59" y="68.58" extent="1-16" drill="0.45"/>
+<via x="33.02" y="34.29" extent="1-16" drill="0.45"/>
+<via x="13.97" y="35.56" extent="1-16" drill="0.45"/>
+<via x="5.08" y="11.43" extent="1-16" drill="0.45"/>
+<via x="31.75" y="8.89" extent="1-16" drill="0.45"/>
+<via x="16.51" y="17.78" extent="1-16" drill="0.45"/>
+<via x="16.51" y="8.89" extent="1-16" drill="0.45"/>
+<via x="7.62" y="41.91" extent="1-16" drill="0.45"/>
+<via x="3.81" y="69.85" extent="1-16" drill="0.45"/>
 </signal>
 <signal name="DIN">
@@
 </drawing>
 <compatibility>
+<note version="6.3" minversion="6.2.2" severity="warning">
+Since Version 6.2.2 text objects can contain more than one line,
+which will not be processed correctly with this version.
+</note>
 <note version="8.2" severity="warning">
 Since Version 8.2, EAGLE supports online libraries. The ids
