File: Transmitter_11-16.brd (EAGLE design)
At the start: 49.2 x 63.5 mm, 23 parts, among them IC1 7805T, IC2 REG1117, IC3 HT12E", M2 WIRELESS-XY-FST#V, Q1 16MHz, U1 328P

Commit message: Add files via upload
Parts:
- renumbered IC1 to V_REG_5, IC2 to V_REG_3.3, IC3 to ENCODER, JP1 to BATTERY, M2 to 433HMZ_TX, U1 to ATMEGA_328

Commit message: Add files via upload
Other:
- board text added: "Team 04 Ver.2"
- board text removed: "Team 04"
Changed lines of the file:
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@@
 <wire x1="49.2" y1="63.49" x2="0" y2="63.49" width="0" layer="20"/>
 <wire x1="0" y1="63.49" x2="0" y2="0" width="0" layer="20"/>
-<text x="7.62" y="33.02" size="1.778" layer="22" font="vector" ratio="15" rot="R90">Team 04</text>
+<text x="48.26" y="38.1" size="1.778" layer="21" font="vector" ratio="15" rot="R90">Team 04
+Ver.2</text>
 </plain>
 <attributes>
@@
 </polygon>
 <via x="15.24" y="35.56" extent="1-16" drill="0.45"/>
-<via x="45.72" y="38.1" extent="1-16" drill="0.45"/>
+<via x="40.64" y="38.1" extent="1-16" drill="0.45"/>
 <via x="5.08" y="38.1" extent="1-16" drill="0.45"/>
 <via x="10.16" y="12.7" extent="1-16" drill="0.45"/>
@@
 </drawing>
 <compatibility>
+<note version="6.3" minversion="6.2.2" severity="warning">
+Since Version 6.2.2 text objects can contain more than one line,
+which will not be processed correctly with this version.
+</note>
 <note version="8.2" severity="warning">
 Since Version 8.2, EAGLE supports online libraries. The ids
